Commit message: Added GpsFix msg -- my bad Bryanna

File: nu_urc_description/urdf/nu_urc_rover.urdf (robot description, URDF)
Before this commit: robot nu_urc_rover, 21 links, 20 joints
Links:
- added link bl_wheel; visual cylinder length=0.1016 radius=0.1016
- added link bl_wheel_shaft; visual box size=0.025 0.025 0.1
- added link br_wheel; visual cylinder length=0.1016 radius=0.1016
- added link br_wheel_shaft; visual box size=0.025 0.025 0.1
- added link fl_wheel; visual cylinder length=0.1016 radius=0.1016
- added link fl_wheel_shaft; visual box size=0.025 0.025 0.1
- added link fr_wheel; visual cylinder length=0.1016 radius=0.1016
- added link fr_wheel_shaft; visual box size=0.025 0.025 0.1
Joints:
- added joint bl_shaft_joint: type continuous, parent bl_chassis, child bl_wheel_shaft, origin xyz=-0.2625 0.0625 0.0 rpy=0.0 0.0 0.0
- added joint bl_wheel_joint: type continuous, parent bl_wheel_shaft, child bl_wheel, origin xyz=0.0 0.1008 0.0 rpy=0.0 0.0 0.0
- added joint br_shaft_joint: type continuous, parent br_chassis, child br_wheel_shaft, origin xyz=-0.2625 -0.0625 0.0 rpy=0.0 0.0 0.0
- added joint br_wheel_joint: type continuous, parent br_wheel_shaft, child br_wheel, origin xyz=0.0 -0.1008 0.0 rpy=0.0 0.0 0.0
- added joint fl_shaft_joint: type continuous, parent bl_chassis, child fl_wheel_shaft, origin xyz=0.2625 0.0625 0.0 rpy=0.0 0.0 0.0
- added joint fl_wheel_joint: type continuous, parent fl_wheel_shaft, child fl_wheel, origin xyz=0.0 0.1008 0.0 rpy=0.0 0.0 0.0
- added joint fr_shaft_joint: type continuous, parent br_chassis, child fr_wheel_shaft, origin xyz=0.2625 -0.0625 0.0 rpy=0.0 0.0 0.0
- added joint fr_wheel_joint: type continuous, parent fr_wheel_shaft, child fr_wheel, origin xyz=0.0 -0.1008 0.0 rpy=0.0 0.0 0.0
- joint base_link_bb_chassis_connector: type fixed -> continuous
- joint base_link_bbl_cube_chassis_connector: type fixed -> continuous
- joint base_link_bbr_cube_chassis_connector: type fixed -> continuous
- joint base_link_bf_chassis_connector: type fixed -> continuous
- joint base_link_bfl_cube_chassis_connector: type fixed -> continuous
- joint base_link_bfr_cube_chassis_connector: type fixed -> continuous
- joint base_link_bl_chassis_connector: type fixed -> continuous
- joint base_link_br_chassis_connector: type fixed -> continuous
- joint bbl_cube_chassis_bt_bl_chassis_connector: type fixed -> continuous
- joint bbr_cube_chassis_bt_br_chassis_connector: type fixed -> continuous
- joint bfl_cube_chassis_bt_fl_chassis_connector: type fixed -> continuous
- joint bfr_cube_chassis_bt_fr_chassis_connector: type fixed -> continuous
- joint bt_bl_chassis_tbl_cube_chassis_connector: type fixed -> continuous
- joint bt_br_chassis_tbr_cube_chassis_connector: type fixed -> continuous
- joint bt_fl_chassis_tfl_cube_chassis_connector: type fixed -> continuous
- joint bt_fr_chassis_tfr_cube_chassis_connector: type fixed -> continuous
- joint tbl_cube_chassis_tb_chassis_connector: type fixed -> continuous
- joint tbl_cube_chassis_tl_chassis_connector: type fixed -> continuous
- joint tfr_cube_chassis_tf_chassis_connector: type fixed -> continuous
- joint tfr_cube_chassis_tr_chassis_connector: type fixed -> continuous

File: nu_urc_description/urdf/nu_urc_rover.xacro (robot description, xacro)
@@ -16,4 +16,8 @@
   <xacro:property name="chassis_z_bottom_dist" value="${(sheet_metal_thickness + cube_length)/2}" />
   <xacro:property name="chassis_z_top_dist" value="${(cube_length + aluminum_bar_length)/2}" />
+  <!-- Wheel properties -->
+  <xacro:property name="wheel_shaft_length" value="0.1" />
+  <xacro:property name="wheel_radius" value="0.1016" />
+  <xacro:property name="wheel_length" value="0.1016" />
   <!--                              BEGIN MACRO DEFINITION                              -->
   <!-- Perforated sheet metal -->
@@ -105,4 +109,50 @@
       <parent link="${parent_base}" />
       <child link="${child_base}" />
+      <origin xyz="${xyz}" rpy="${rpy}" />
+    </joint>
+  </xacro:macro>
+  <xacro:macro name="rover_transmission" params="short_name long_name">
+    <transmission name="${short_name}_transmission">
+      <type>transmission_interface/SimpleTransmission</type>
+      <joint name="${short_name}_wheel_joint">
+        <hardwareInterface>EffortJointInterface</hardwareInterface>
+      </joint>
+      <actuator name="${long_name}">
+        <hardwareInterface>EffortJointInterface</hardwareInterface>
+        <mechanicalReduction>1</mechanicalReduction>
+      </actuator>
+    </transmission>
+  </xacro:macro>
+  <xacro:macro name="wheel_shaft" params="name bar_length cs_length">
+    <link name="${name}_wheel_shaft">
+      <visual>
+        <geometry>
+          <box size="${cs_length} ${cs_length} ${bar_length}" />
+        </geometry>
+        <origin rpy="1.570796 0.0 0.0" xyz="0.0 0.0 0.0" />
+      </visual>
+    </link>
+  </xacro:macro>
+  <xacro:macro name="wheel" params="name radius length">
+    <link name="${name}_wheel">
+      <visual>
+        <geometry>
+          <cylinder radius="${radius}" length="${length}" />
+        </geometry>
+        <origin xyz="0.0 0.0 0.0" rpy="1.570796 0.0 0.0" />
+      </visual>
+    </link>
+  </xacro:macro>
+  <xacro:macro name="chassis_shaft_joint" params="exta_name shaft_name xyz rpy">
+    <joint name="${shaft_name}_shaft_joint" type="continuous">
+      <parent link="${exta_name}_chassis" />
+      <child link="${shaft_name}_wheel_shaft" />
+      <origin xyz="${xyz}" rpy="${rpy}" />
+    </joint>
+  </xacro:macro>
+  <xacro:macro name="shaft_wheel_joint" params="wheel_name shaft_name xyz rpy">
+    <joint name="${wheel_name}_wheel_joint" type="continuous">
+      <parent link="${shaft_name}_wheel_shaft" />
+      <child link="${wheel_name}_wheel" />
       <origin xyz="${xyz}" rpy="${rpy}" />
     </joint>
@@ -135,5 +185,14 @@
   <xacro:cube_connector name="bbl_cube_chassis" length="${cube_length}" />
   <xacro:cube_connector name="bbr_cube_chassis" length="${cube_length}" />
-  <!--                               END LINK DEFINITION                              -->
+  <!-- Generate all the wheel and associated links -->
+  <xacro:wheel_shaft name="fl" bar_length="${wheel_shaft_length}" cs_length="${aluminum_cs_length}" />
+  <xacro:wheel_shaft name="fr" bar_length="${wheel_shaft_length}" cs_length="${aluminum_cs_length}" />
+  <xacro:wheel_shaft name="bl" bar_length="${wheel_shaft_length}" cs_length="${aluminum_cs_length}" />
+  <xacro:wheel_shaft name="br" bar_length="${wheel_shaft_length}" cs_length="${aluminum_cs_length}" />
+  <xacro:wheel name="fl" radius="${wheel_radius}" length="${wheel_length}" />
+  <xacro:wheel name="fr" radius="${wheel_radius}" length="${wheel_length}" />
+  <xacro:wheel name="bl" radius="${wheel_radius}" length="${wheel_length}" />
+  <xacro:wheel name="br" radius="${wheel_radius}" length="${wheel_length}" />
+  <!--                              END LINK DEFINITION                              -->
   <!--                              BEGIN JOINT DEFINITION                              -->
   <!-- Base link bottom connections -->
@@ -161,4 +220,18 @@
   <xacro:chassis_generation parent_base="tbl_cube_chassis" child_base="tb_chassis" xyz="0.0 -${chassis_y_dist} 0.0" rpy="0.0 0.0 0.0" />
   <xacro:chassis_generation parent_base="tbl_cube_chassis" child_base="tl_chassis" xyz="${chassis_x_dist} 0.0 0.0" rpy="0.0 0.0 0.0" />
+  <!-- All of the wheel joints -->
+  <xacro:chassis_shaft_joint shaft_name="fl" exta_name="bl" xyz="${(aluminum_bar_length-aluminum_cs_length)/2} ${(wheel_shaft_length+aluminum_cs_length)/2} 0.0" rpy="0.0 0.0 0.0" />
+  <xacro:chassis_shaft_joint shaft_name="fr" exta_name="br" xyz="${(aluminum_bar_length-aluminum_cs_length)/2} -${(wheel_shaft_length+aluminum_cs_length)/2} 0.0" rpy="0.0 0.0 0.0" />
+  <xacro:chassis_shaft_joint shaft_name="bl" exta_name="bl" xyz="-${(aluminum_bar_length-aluminum_cs_length)/2} ${(wheel_shaft_length+aluminum_cs_length)/2} 0.0" rpy="0.0 0.0 0.0" />
+  <xacro:chassis_shaft_joint shaft_name="br" exta_name="br" xyz="-${(aluminum_bar_length-aluminum_cs_length)/2} -${(wheel_shaft_length+aluminum_cs_length)/2} 0.0" rpy="0.0 0.0 0.0" />
+  <xacro:shaft_wheel_joint wheel_name="fl" shaft_name="fl" xyz="0.0 ${(wheel_shaft_length+wheel_length)/2} 0.0" rpy="0.0 0.0 0.0" />
+  <xacro:shaft_wheel_joint wheel_name="fr" shaft_name="fr" xyz="0.0 ${-(wheel_shaft_length+wheel_length)/2} 0.0" rpy="0.0 0.0 0.0" />
+  <xacro:shaft_wheel_joint wheel_name="bl" shaft_name="bl"  xyz="0.0 ${(wheel_shaft_length+wheel_length)/2} 0.0" rpy="0.0 0.0 0.0" />
+  <xacro:shaft_wheel_joint wheel_name="br" shaft_name="br" xyz="0.0 ${-(wheel_shaft_length+wheel_length)/2} 0.0" rpy="0.0 0.0 0.0" />
   <!--                               END JOINT DEFINITION                              -->
+  <!--                           BEGIN MOTOR TRANSMISSION DEFINITION                   -->
+  <xacro:rover_transmission short_name="fl" long_name="front_left" />
+  <xacro:rover_transmission short_name="fr" long_name="front_right" />
+  <xacro:rover_transmission short_name="bl" long_name="back_left" />
+  <xacro:rover_transmission short_name="br" long_name="back_right" />
 </robot>
