Commit message: Added first prototype of arm model

File: nu_urc_description/urdf/nu_urc_arm.urdf (robot description, URDF)
Before this commit: robot nu_urc_arm, 4 links, 3 joints
Links:
- link arm_prism_base: geometry visual box size=0.1016 0.4572 0.1016
- link arm_swivel_base: geometry visual box size=0.1016 0.1016 0.1016
Joints:
- joint arm_prism_base_swivel_base: origin xyz=0.0 0.0 1 rpy=0.0 0.0 0.0 -> xyz=0.0 0.0 0.1016 rpy=0.0 0.0 0.0
- joint arm_swivel_base_rot_0: origin xyz=0.0 0.0 0.0254 rpy=0.0 0.0 0.0 -> xyz=0.0 0.0 0.0508 rpy=0.0 0.0 0.0

File: nu_urc_description/urdf/nu_urc_arm.xacro (robot description, xacro)
@@ -4,11 +4,11 @@
 <xacro:property name="pi" value="3.1415926" />
 <!-- The dimensions of the arm base's linear rail system -->
-<xacro:property name="arm_prism_base_l" value="1" />
-<xacro:property name="arm_prism_base_w" value="1" />
-<xacro:property name="arm_prism_base_h" value="1" />
+<xacro:property name="arm_prism_base_l" value="0.4572" />
+<xacro:property name="arm_prism_base_w" value="0.1016" />
+<xacro:property name="arm_prism_base_h" value="0.1016" />
 <!-- The dimensions of the arm base's swivel system -->
-<xacro:property name="arm_swivel_base_l" value="1" />
-<xacro:property name="arm_swivel_base_w" value="1" />
-<xacro:property name="arm_swivel_base_h" value="1" />
+<xacro:property name="arm_swivel_base_l" value="0.1016" />
+<xacro:property name="arm_swivel_base_w" value="0.1016" />
+<xacro:property name="arm_swivel_base_h" value="0.1016" />
 <!-- The dimensions of first arm link -->
 <!-- The two revolute arm links are the same length at around 9.5 inches -->
@@ -22,5 +22,6 @@
 <xacro:property name="arm_rot_1_h" value="0.0381" />
 <!-- The displacement of first arm link with respect to the swivel base -->
-<xacro:property name="arm_swivel_base_rot_0_h" value="0.0254" />
+<xacro:property name="arm_prism_base_swivel_base_h" value="${(arm_prism_base_h+arm_swivel_base_h)/2}" />
+<xacro:property name="arm_swivel_base_rot_0_h" value="${arm_swivel_base_h/2}" />
 <!-- Joint Limits -->
 <xacro:property name="arm_swivel_base_rot_0_lower" value="0" />
@@ -31,5 +32,5 @@
   <visual>
     <geometry>
-      <box size="${arm_prism_base_w} ${arm_prism_base_h} ${arm_prism_base_l}" />
+      <box size="${arm_prism_base_w} ${arm_prism_base_l} ${arm_prism_base_h}" />
       <origin rpy="0.0 0.0 0.0" xyz="0.0 0.0 0.0" />
     </geometry>
@@ -48,6 +49,6 @@
     <geometry>
       <box size="${arm_rot_0_w} ${arm_rot_0_h} ${arm_rot_0_l}" />
-      <origin rpy="0.0 0.0 0.0" xyz="0.0 0.0 0.0" />
     </geometry>
+   <origin rpy="0.0 0.0 0.0" xyz="0.0 0.0 ${arm_rot_0_l/2}" />
   </visual>
 </link>
@@ -56,6 +57,6 @@
     <geometry>
       <box size="${arm_rot_1_w} ${arm_rot_1_h} ${arm_rot_1_l}" />
-      <origin rpy="0.0 0.0 0.0" xyz="0.0 0.0 0.0" />
     </geometry>
+    <origin rpy="0.0 0.0 0.0" xyz="0.0 0.0 ${arm_rot_1_l/2}" />
   </visual>
 </link>
@@ -63,5 +64,5 @@
   <parent link="arm_prism_base" />
   <child link="arm_swivel_base" />
-  <origin xyz="0.0 0.0 ${arm_prism_base_h}" rpy="0.0 0.0 0.0" />
+  <origin xyz="0.0 0.0 ${arm_prism_base_swivel_base_h}" rpy="0.0 0.0 0.0" />
   <axis xyz="0 0 1" />
 </joint>
